File: hardware/vomit_light_v1.kicad_sch (KiCad schematic)
At the start: 19 parts, among them K1 SPDT, K2 SPDT, K3 SPDT, P1 Conn_WallPlug

Commit message: schematic updates
Connections:
- net RETURN_WLED_1 renamed GND_WLED_1
- net RETURN_WLED_2 renamed GND_WLED_2
- new net: RGB5. (VSS), RGB6. (VSS) (x2)
- new net: RGB4. (VSS), RGB5. (VSS) (x2)
- new net: RGB1. (VSS), RGB2. (VSS) (x2)
- new net: RGB3. (VSS), RGB4. (VSS) (x2)
- new net: RGB2. (VSS), RGB3. (VSS) (x2)
Other:
- moved on the sheet: D1, D2, D3, D4, D5, D6, K2, K3, PS2, PS3, RGB1, RGB2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

Commit message: v1 schematic done
Parts:
- added J1, J2: Wire, symbol Connector_Generic:Conn_01x01
- added RGB10, RGB11, RGB12, RGB7, RGB8, RGB9: WS2801 Strip xN, symbol vomit_light:WS2801_strip
- added U1: Arduino, symbol Connector_Generic:Conn_01x06
Connections:
- net +5V: now also J1.1 (Pin_1); no longer RGB1. (VSS), RGB2. (VSS), RGB3. (VSS), RGB4. (VSS), RGB5. (VSS), RGB6. (VSS)
- net 5V_OUT: now also RGB1. (DO), RGB2. (DO), RGB3. (DO), RGB4. (DO), RGB5. (DO), RGB6. (DO), RGB10. (DO), RGB11. (DO), RGB12. (DO), RGB7. (DO), RGB8. (DO), RGB9. (DO), U1.5 (Pin_5)
- net GND: now also RGB10. (DO), RGB11. (DO), RGB12. (DO), RGB7. (DO), RGB8. (DO), RGB9. (DO), U1.6 (Pin_6)
- net RELAY_9_RETURN: now also J2.1 (Pin_1)
- net SPI1_SCLK: now reaches RGB1. (DO)
- net SPI1_SCLK: now also U1.4 (Pin_4)
- net AC_L: now reaches P1.1 (AC_P), PS1.1 (AC/L), PS2.1 (AC/L), PS3.1 (AC/L)
- net AC_N: now reaches P1.2 (AC_N), PS1.2 (AC/N), PS2.2 (AC/N), PS3.2 (AC/N)
- net GND_WLED_1: no longer names the net of D1.1 (K), D2.1 (K), D3.1 (K), K2.COM
- net GND_WLED_2: no longer names the net of D4.1 (K), D5.1 (K), D6.1 (K), K3.COM
- new net: RGB7. (DO), RGB8. (DO) (x2)
- new net: RGB8. (DO), RGB9. (DO) (x2)
- new net: RGB10. (DO), RGB11. (DO) (x2)
- new net: RGB10. (DO), RGB9. (DO) (x2)
- new net: RGB11. (DO), RGB12. (DO) (x2)
- new net: RGB1. (DO), RGB2. (DO) (x2)
- new net: RGB3. (DO), RGB4. (DO) (x2)
- new net: RGB4. (DO), RGB5. (DO) (x2)
- new net: RGB2. (DO), RGB3. (DO) (x2)
- new net: RGB5. (DO), RGB6. (DO) (x2)
- new net SPI0_MOSI: RGB7. (DO), U1.1 (Pin_1)
- new net SPI0_SCLK: RGB7. (DO), U1.2 (Pin_2)
- new net SPI1_MOSI: RGB1. (DO), U1.3 (Pin_3)
- no-connect marks 3 -> 7
Other:
- note added: "Controller"
- note added: "Power Supplies"
- note added: "RGB LED Strips"
- note added: "White LEDs"
- moved on the sheet: D1, D2, D3, D4, D5, D6, K1, K2, K3, P1, PS1, PS2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
