File: hardware/v2/vomit_light_v2.kicad_sch (KiCad schematic)
At the start: 28 parts, among them J1 Wire, J2 Wire, K1 SPDT, K2 SPDT, K3 SPDT, P1 Conn_WallPlug, U1 Arduino

Commit message: V2 schematic check in
Parts:
- removed U1: Arduino, symbol Connector_Generic:Conn_01x06
Connections:
- new net: RGB7. (DO), RGB8. (DO) (x2)
- new net: RGB8. (DO), RGB9. (DO) (x2)
- new net: RGB10. (DO), RGB11. (DO) (x2)
- new net: RGB10. (DO), RGB9. (DO) (x2)
- new net: RGB11. (DO), RGB12. (DO) (x2)
- new net: RGB1. (DO), RGB2. (DO) (x2)
- new net: RGB3. (DO), RGB4. (DO) (x2)
- new net: RGB4. (DO), RGB5. (DO) (x2)
- new net: RGB2. (DO), RGB3. (DO) (x2)
- new net: RGB5. (DO), RGB6. (DO) (x2)
Other:
- added sheet control_board (control_board.kicad_sch)
- moved on the sheet: J1, J2, K1, P1, PS1, PS2, PS3
