File: hardware/v2/_autosave-vomit_light_v2.kicad_sch (KiCad schematic)
At the start: 4 parts, among them J1 Screw_Terminal_01x03, J2 Screw_Terminal_01x03, J3 Screw_Terminal_01x03, U1 RP PICO

Commit message: schematic check in
Parts:
- added J4, J5: Screw_Terminal_01x03, symbol Connector:Screw_Terminal_01x03
Connections:
- net GND: now also J4.1 (Pin_1), J5.3 (Pin_3)
- net SPARE3: now also U1.19 (GPIO14), J5.1 (Pin_1)
- net SPARE4: now reaches U1.20 (GPIO15)
- net SPARE4: now also J5.2 (Pin_2)
- net SPI0_MOSI renamed RGB1_DAT
- net RGB1_DAT: now also J4.3 (Pin_3)
- net SPI0_SCLK renamed RGB1_CLK
- net RGB1_CLK: now also J4.2 (Pin_2)
Changed lines of the file:
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@@
+    (stroke (width 0) (type default))
+  )
+  (wire (pts (xy 124.46 142.24) (xy 127 142.24))
     (stroke (width 0) (type default))
   )
@@
     (stroke (width 0) (type default))
   )
+  (wire (pts (xy 101.6 137.16) (xy 127 137.16))
+    (stroke (width 0) (type default))
+  )
   (wire (pts (xy 121.92 132.08) (xy 121.92 124.46))
     (stroke (width 0) (type default))
@@
     (stroke (width 0) (type default))
   )
+  (wire (pts (xy 121.92 147.32) (xy 127 147.32))
+    (stroke (width 0) (type default))
+  )
   (wire (pts (xy 219.71 127) (xy 219.71 124.46))
     (stroke (width 0) (type default))
@@
     (stroke (width 0) (type default))
   )
-  (wire (pts (xy 101.6 149.86) (xy 109.22 149.86))
+  (wire (pts (xy 101.6 149.86) (xy 127 149.86))
     (stroke (width 0) (type default))
   )
@@
     (stroke (width 0) (type default))
   )
+  (wire (pts (xy 101.6 139.7) (xy 127 139.7))
+    (stroke (width 0) (type default))
+  )
   (wire (pts (xy 124.46 114.3) (xy 127 114.3))
     (stroke (width 0) (type default))
@@
     (stroke (width 0) (type default))
   )
-  (wire (pts (xy 109.22 152.4) (xy 101.6 152.4))
+  (wire (pts (xy 101.6 152.4) (xy 127 152.4))
     (stroke (width 0) (type default))
   )
@@
     (stroke (width 0) (type default))
   )
+  (wire (pts (xy 121.92 154.94) (xy 121.92 147.32))
+    (stroke (width 0) (type default))
+  )
   (wire (pts (xy 222.25 127) (xy 219.71 127))
     (stroke (width 0) (type default))
@@
   )
   (label "5V_OUT" (at 222.25 127 0) (fields_autoplaced)
+    (effects (font (size 1.27 1.27)) (justify left bottom))
+  )
+  (label "SPARE3" (at 116.84 137.16 0) (fields_autoplaced)
+    (effects (font (size 1.27 1.27)) (justify left bottom))
+  )
+  (label "RGB1_DAT" (at 106.68 152.4 0) (fields_autoplaced)
+    (effects (font (size 1.27 1.27)) (justify left bottom))
+  )
+  (label "RGB1_CLK" (at 106.68 149.86 0) (fields_autoplaced)
+    (effects (font (size 1.27 1.27)) (justify left bottom))
+  )
+  (label "SPARE4" (at 116.84 139.7 0) (fields_autoplaced)
     (effects (font (size 1.27 1.27)) (justify left bottom))
   )
@@
     (effects (font (size 1.27 1.27)) (justify left))
   )
-  (hierarchical_label "SPI0_SCLK" (shape output) (at 109.22 149.86 0) (fields_autoplaced)
-    (effects (font (size 1.27 1.27)) (justify left))
-  )
   (hierarchical_label "SPARE0" (shape bidirectional) (at 157.48 93.98 0) (fields_autoplaced)
-    (effects (font (size 1.27 1.27)) (justify left))
-  )
-  (hierarchical_label "SPI0_MOSI" (shape output) (at 109.22 152.4 0) (fields_autoplaced)
     (effects (font (size 1.27 1.27)) (justify left))
   )
@@
       (effects (font (size 1.27 1.27)) hide)
     )
-    (property "Value" "GND" (at 116.84 134.62 0)
+    (property "Value" "GND" (at 119.38 132.08 0)
       (effects (font (size 1.27 1.27)))
     )
@@
     )
   )
+  (symbol (lib_id "Connector:Screw_Terminal_01x03") (at 132.08 139.7 0) (unit 1)
+    (in_bom yes) (on_board yes) (dnp no) (fields_autoplaced)
+    (property "Reference" "J5" (at 134.62 139.065 0)
+      (effects (font (size 1.27 1.27)) (justify left))
+    )
+    (property "Value" "Screw_Terminal_01x03" (at 134.62 141.605 0)
+      (effects (font (size 1.27 1.27)) (justify left) hide)
+    )
+    (property "Footprint" "" (at 132.08 139.7 0)
+      (effects (font (size 1.27 1.27)) hide)
+    )
+    (property "Datasheet" "~" (at 132.08 139.7 0)
+      (effects (font (size 1.27 1.27)) hide)
+    )
+    (pin "1")
+    (pin "2")
+    (pin "3")
+    (instances
+      (project "vomit_light_v2"
+        (path "/f4f0a6e0-0d7b-4662-b4bd-fb29ae5fadd3"
+          (reference "J5") (unit 1)
+        )
+      )
+    )
+  )
+  (symbol (lib_id "Connector:Screw_Terminal_01x03") (at 132.08 149.86 0) (unit 1)
+    (in_bom yes) (on_board yes) (dnp no) (fields_autoplaced)
+    (property "Reference" "J4" (at 134.62 149.225 0)
+      (effects (font (size 1.27 1.27)) (justify left))
+    )
+    (property "Value" "Screw_Terminal_01x03" (at 134.62 151.765 0)
+      (effects (font (size 1.27 1.27)) (justify left) hide)
+    )
+    (property "Footprint" "" (at 132.08 149.86 0)
+      (effects (font (size 1.27 1.27)) hide)
+    )
+    (property "Datasheet" "~" (at 132.08 149.86 0)
+      (effects (font (size 1.27 1.27)) hide)
+    )
+    (pin "1")
+    (pin "2")
+    (pin "3")
+    (instances
+      (project "vomit_light_v2"
+        (path "/f4f0a6e0-0d7b-4662-b4bd-fb29ae5fadd3"
+          (reference "J4") (unit 1)
+        )
+      )
+    )
+  )
+  (symbol (lib_id "power:GND") (at 124.46 142.24 0) (unit 1)
+    (in_bom yes) (on_board yes) (dnp no)
+    (property "Reference" "#PWR05" (at 124.46 148.59 0)
+      (effects (font (size 1.27 1.27)) hide)
+    )
+    (property "Value" "GND" (at 121.92 142.24 0)
+      (effects (font (size 1.27 1.27)))
+    )
+    (property "Footprint" "" (at 124.46 142.24 0)
+      (effects (font (size 1.27 1.27)) hide)
+    )
+    (property "Datasheet" "" (at 124.46 142.24 0)
+      (effects (font (size 1.27 1.27)) hide)
+    )
+    (pin "1")
+    (instances
+      (project "vomit_light_v2"
+        (path "/f4f0a6e0-0d7b-4662-b4bd-fb29ae5fadd3"
+          (reference "#PWR05") (unit 1)
+        )
+      )
+    )
+  )
   (symbol (lib_id "power:GND") (at 124.46 114.3 0) (unit 1)
     (in_bom yes) (on_board yes) (dnp no)
@@
         )
       )
+    )
+  )
+  (symbol (lib_id "power:GND") (at 121.92 154.94 0) (unit 1)
+    (in_bom yes) (on_board yes) (dnp no)
+    (property "Reference" "#PWR04" (at 121.92 161.29 0)
+      (effects (font (size 1.27 1.27)) hide)
+    )
+    (property "Value" "GND" (at 116.84 154.94 0)
+      (effects (font (size 1.27 1.27)))
+    )
+    (property "Footprint" "" (at 121.92 154.94 0)
+      (effects (font (size 1.27 1.27)) hide)
+    )
+    (property "Datasheet" "" (at 121.92 154.94 0)
+      (effects (font (size 1.27 1.27)) hide)
+    )
+    (pin "1")
+    (instances
+      (project "vomit_light_v2"
+        (path "/f4f0a6e0-0d7b-4662-b4bd-fb29ae5fadd3"
+          (reference "#PWR04") (unit 1)
+        )
+      )
